File: kicad project/sym5v/sym5v.sch (KiCad schematic (older format))
At the start: 31 parts

Commit message: Rev1
Parts:
- removed C? (x2): C, symbol Device:C
- added C11, C4: 47uF, Capacitor_SMD:CP_Elec_6.3x5.8, symbol Device:CP1
- added J2: Conn_01x03, Connector_Wire:SolderWirePad_1x03_P3.81mm_Drill1.2mm, symbol Connector_Generic:Conn_01x03
- added U4: TUSB321AI, symbol LoaDy:TUSB321AI
- C1, C10, C12, C13, C14, C15, C16, C17, C18, C3: renamed from C?; footprint (none) -> Capacitor_SMD:C_1210_3225Metric
- C2, C5, C6, C7, C8, C9: renamed from C?; footprint (none) -> Capacitor_SMD:C_0603_1608Metric
- D1, D2: renamed from D?; footprint (none) -> LoaDy:DO-214AC
- J1: renamed from J?; footprint (none) -> Connector_USB:USB_C_Receptacle_Amphenol_12401548E4-2A
- L1, L2: renamed from L?; footprint (none) -> Inductor_SMD:L_7.3x7.3_H3.5
- R1, R2, R5: renamed from R?; footprint (none) -> Resistor_SMD:R_0603_1608Metric
- R3: renamed from R?; value 680K -> 665K; footprint (none) -> Resistor_SMD:R_0603_1608Metric
- R4: renamed from R?; value 562K -> 536K; footprint (none) -> Resistor_SMD:R_0603_1608Metric
- U1: renamed from U?; footprint (none) -> Package_DFN_QFN:QFN-24-1EP_4x4mm_P0.5mm_EP2.6x2.6mm
- U2: renamed from U?; footprint (none) -> Package_TO_SOT_SMD:TO-263-3_TabPin4
- U3: renamed from U?; footprint (none) -> Package_TO_SOT_SMD:TO-263-3_TabPin2
Connections:
- wire segments 152 -> 159
- no-connect marks 16 -> 15
Other:
- note added: "VNEG set to about -6.21V"
- note added: "VPOS set to about 6.21V"
- note removed: "Current capability detection here\n\nType-C can do 1.5A or 3A @ 5V by default without PD\nUp to 20V 5A with PD - requires complicated\nPD chips and solutions\n\nSimple ICs exist to detect current capability \nof source -> LOW/HIGH current \nsignalisation (TI TUSB321AI)"
- note removed: "VNEG set to about -6.35V"
- note removed: "VPOS set to about 6.45V"

Commit message: Rev 2 schematic - broken symbols!
Parts:
- added R6: 100K, Resistor_SMD:R_0603_1608Metric, symbol Device:R_Small
- C11, C4: footprint Capacitor_SMD:CP_Elec_6.3x5.8 -> Capacitor_Tantalum_SMD:CP_EIA-7343-31_Kemet-D_Pad2.25x2.55mm_HandSolder
Connections:
- wire segments 159 -> 160
Other:
- note added: "Output LDO Regulators"
- note added: "Split-rail DC/DC Converter"
- note added: "USB C Connection"
- note added: "USB-C power delivery chip not used"
