File: kicad project/sym5v.kicad_pcb (KiCad board)
At the start: 2 copper layers, 80.8 x 30.5 mm, 33 parts, among them J1 USB_C_Receptacle, J2 Conn_01x03, U1 TPS6513x, U2 LM2940, U3 LM2990SX-5.0

Commit message: add mounting holes
Parts:
- added ?: MountingHole_3.2mm_M3_ISO14580, MountingHole:MountingHole_3.2mm_M3_ISO14580, F.Cu at (78.1, 87.2)
- added ?: MountingHole_3.2mm_M3_ISO14580, MountingHole:MountingHole_3.2mm_M3_ISO14580, F.Cu at (153.2, 112.0)
Routing:
- net GND: vias 72 -> 68
Changed lines of the file:
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@@
     (thickness 1.6)
     (drawings 12)
-    (tracks 176)
+    (tracks 172)
     (zones 0)
-    (modules 33)
+    (modules 35)
     (nets 35)
   )
@@
   )
   (setup
-    (last_trace_width 2.5)
+    (last_trace_width 0.2)
     (user_trace_width 0.3)
     (user_trace_width 0.5)
@@
     (add_net VPOS)
   )
+  (module MountingHole:MountingHole_3.2mm_M3_ISO14580 (layer F.Cu)
+    (at 78.105 87.249)
+    (descr "Mounting Hole 3.2mm, no annular, M3, ISO14580")
+    (tags "mounting hole 3.2mm no annular m3 iso14580")
+    (attr virtual)
+    (fp_text reference "" (at 0 -3.75) (layer F.SilkS)
+      (effects (font (size 1 1) (thickness 0.15)))
+    )
+    (fp_text value MountingHole_3.2mm_M3_ISO14580 (at 0 -4.191) (layer F.Fab)
+      (effects (font (size 1 1) (thickness 0.15)))
+    )
+    (fp_text user %R (at 0.3 0) (layer F.Fab)
+      (effects (font (size 1 1) (thickness 0.15)))
+    )
+    (fp_circle (center 0 0) (end 2.75 0) (layer Cmts.User) (width 0.15))
+    (fp_circle (center 0 0) (end 3 0) (layer F.CrtYd) (width 0.05))
+    (pad 1 np_thru_hole circle (at 0 0) (size 3.2 3.2) (drill 3.2) (layers *.Cu *.Mask))
+  )
   (module Capacitor_Tantalum_SMD:CP_EIA-7343-31_Kemet-D_Pad2.25x2.55mm_HandSolder (layer F.Cu)
     (at 88.392 90.399 270)
@@
     )
   )
+  (module MountingHole:MountingHole_3.2mm_M3_ISO14580 (layer F.Cu)
+    (at 153.162 112.014)
+    (descr "Mounting Hole 3.2mm, no annular, M3, ISO14580")
+    (tags "mounting hole 3.2mm no annular m3 iso14580")
+    (attr virtual)
+    (fp_text reference "" (at 0 -3.75) (layer F.SilkS)
+      (effects (font (size 1 1) (thickness 0.15)))
+    )
+    (fp_text value MountingHole_3.2mm_M3_ISO14580 (at 0 3.75) (layer F.Fab)
+      (effects (font (size 1 1) (thickness 0.15)))
+    )
+    (fp_circle (center 0 0) (end 3 0) (layer F.CrtYd) (width 0.05))
+    (fp_circle (center 0 0) (end 2.75 0) (layer Cmts.User) (width 0.15))
+    (fp_text user %R (at 0.3 0) (layer F.Fab)
+      (effects (font (size 1 1) (thickness 0.15)))
+    )
+    (pad 1 np_thru_hole circle (at 0 0) (size 3.2 3.2) (drill 3.2) (layers *.Cu *.Mask))
+  )
   (gr_text GND (at 85.852 97.409) (layer F.SilkS)
     (effects (font (size 2 2) (thickness 0.3)))
@@
     (effects (font (size 1 1) (thickness 0.15)))
   )
-  (gr_text "O. Pecák, FI MUNI, March 2019" (at 143.891 113.792) (layer F.SilkS)
+  (gr_text "O. Pecák, FI MUNI, March 2019" (at 139.319 113.792) (layer F.SilkS)
     (effects (font (size 1 1) (thickness 0.15)))
   )
@@
   (gr_line (start 156.083 114.935) (end 156.083 84.455) (layer Edge.Cuts) (width 0.15))
   (gr_line (start 75.311 84.455) (end 75.311 114.808) (layer Edge.Cuts) (width 0.15))
-  (via (at 101.6 110.871) (size 2) (drill 0.7) (layers F.Cu B.Cu) (net 3))
-  (via (at 98.679 110.871) (size 2) (drill 0.7) (layers F.Cu B.Cu) (net 3))
-  (via (at 95.758 110.871) (size 2) (drill 0.7) (layers F.Cu B.Cu) (net 3))
-  (via (at 95.758 104.394) (size 2) (drill 0.7) (layers F.Cu B.Cu) (net 3))
-  (via (at 98.806 104.394) (size 2) (drill 0.7) (layers F.Cu B.Cu) (net 3))
-  (via (at 101.727 104.394) (size 2) (drill 0.7) (layers F.Cu B.Cu) (net 3))
-  (via (at 95.885 107.696) (size 2) (drill 0.7) (layers F.Cu B.Cu) (net 3))
   (segment (start 135.001 99.695) (end 135.255 99.441) (width 0.3) (layer F.Cu) (net 1))
   (segment (start 135.255 99.441) (end 136.017 99.441) (width 0.3) (layer F.Cu) (net 1))
@@
   (segment (start 146.531 93.275) (end 143.186 93.275) (width 0.5) (layer B.Cu) (net 2))
   (segment (start 143.186 93.275) (end 143.129 93.218) (width 0.5) (layer B.Cu) (net 2))
+  (via (at 101.6 110.871) (size 2) (drill 0.7) (layers F.Cu B.Cu) (net 3))
+  (via (at 98.679 110.871) (size 2) (drill 0.7) (layers F.Cu B.Cu) (net 3))
+  (via (at 95.758 110.871) (size 2) (drill 0.7) (layers F.Cu B.Cu) (net 3))
+  (via (at 95.758 104.394) (size 2) (drill 0.7) (layers F.Cu B.Cu) (net 3))
+  (via (at 98.806 104.394) (size 2) (drill 0.7) (layers F.Cu B.Cu) (net 3))
+  (via (at 101.727 104.394) (size 2) (drill 0.7) (layers F.Cu B.Cu) (net 3))
+  (via (at 95.885 107.696) (size 2) (drill 0.7) (layers F.Cu B.Cu) (net 3))
   (via (at 132.588 100.965) (size 0.8) (drill 0.4) (layers F.Cu B.Cu) (net 3))
   (via (at 132.588 99.949) (size 0.8) (drill 0.4) (layers F.Cu B.Cu) (net 3))
@@
   (via (at 124.46 90.17) (size 2) (drill 0.7) (layers F.Cu B.Cu) (net 3))
   (via (at 139.319 109.982) (size 2) (drill 0.7) (layers F.Cu B.Cu) (net 3))
-  (via (at 152.4 109.982) (size 2) (drill 0.7) (layers F.Cu B.Cu) (net 3))
-  (via (at 150.495 112.522) (size 2) (drill 0.7) (layers F.Cu B.Cu) (net 3))
   (via (at 146.177 112.522) (size 2) (drill 0.7) (layers F.Cu B.Cu) (net 3))
   (via (at 144.018 109.982) (size 2) (drill 0.7) (layers F.Cu B.Cu) (net 3))
@@
   (via (at 83.312 111.887) (size 2) (drill 0.7) (layers F.Cu B.Cu) (net 3))
   (via (at 85.217 109.22) (size 2) (drill 0.7) (layers F.Cu B.Cu) (net 3))
-  (via (at 77.724 90.297) (size 2) (drill 0.7) (layers F.Cu B.Cu) (net 3))
-  (via (at 79.883 87.503) (size 2) (drill 0.7) (layers F.Cu B.Cu) (net 3))
   (via (at 81.915 90.297) (size 2) (drill 0.7) (layers F.Cu B.Cu) (net 3))
   (via (at 86.106 90.297) (size 2) (drill 0.7) (layers F.Cu B.Cu) (net 3))
@@
   (segment (start 79.248 93.599) (end 88.392 93.599) (width 2.5) (layer F.Cu) (net 9))
   (segment (start 88.392 93.599) (end 96.26 93.599) (width 2.5) (layer F.Cu) (net 9))
-  (segment (start 128.0965 101.346) (end 127.559 101.346) (width 0.2) (layer F.Cu) (net 34))
   (segment (start 129.63 101.707) (end 130.1425 101.707) (width 0.2) (layer F.Cu) (net 14))
   (segment (start 129.30501 102.67299) (end 127.635 104.343) (width 0.2) (layer F.Cu) (net 14))
@@
   (segment (start 93.218 99.06) (end 91.059 101.219) (width 2.5) (layer F.Cu) (net 17))
   (segment (start 88.9 101.219) (end 79.248 101.219) (width 2.5) (layer F.Cu) (net 17))
+  (segment (start 128.0965 101.346) (end 127.559 101.346) (width 0.2) (layer F.Cu) (net 34))
   (segment (start 127.7875 101.092) (end 128.651 101.092) (width 0.2) (layer F.Cu) (net 34))
   (segment (start 129.036 100.707) (end 130.1425 100.707) (width 0.2) (layer F.Cu) (net 34))
